File: PCB/PCB_VuilBak_Kicad/_autosave-PCB_VuilBak.kicad_pcb (KiCad board)
At the start: 2 copper layers, 99.9 x 64.2 mm, 39 parts, among them Q1 2N7002, Q2 2N7002, U1 micro_usb, U2 AMS1117-3.3, U3 TCA9548A_I2C_Multiplexer, U4 esp_wroom_32, X1 DG3XX-04-3.5, X10 DG3XX-04-3.5, X11 DG3XX-02-3.5, X12 DG3XX-02-3.5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

Commit message: Update pcb
Changed lines of the file:
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@@
   (segment (start 155.69 71.75) (end 161.4525 71.75) (width 0.5) (layer "B.Cu") (net 5))
   (segment (start 164.4 39.9) (end 164.4 71.5) (width 0.5) (layer "B.Cu") (net 5))
-  (segment (start 175.484 75.184) (end 167.64 75.184) (width 0.254) (layer "B.Cu") (net 6))
+  (segment (start 175.484 75.184) (end 167.64 75.184) (width 0.4) (layer "B.Cu") (net 6))
   (segment (start 142.9 60.7) (end 142.9 69.5) (width 0.5) (layer "B.Cu") (net 6))
-  (segment (start 176.3 77.24) (end 179.832 80.772) (width 0.254) (layer "B.Cu") (net 6))
-  (segment (start 176.3 76) (end 176.3 77.24) (width 0.254) (layer "B.Cu") (net 6))
+  (segment (start 176.3 77.24) (end 179.832 80.772) (width 0.4) (layer "B.Cu") (net 6))
+  (segment (start 176.3 76) (end 176.3 77.24) (width 0.4) (layer "B.Cu") (net 6))
   (segment (start 177.5 83.55) (end 177.48 83.57) (width 0.254) (layer "B.Cu") (net 6))
-  (segment (start 167.64 75.184) (end 166.824 76) (width 0.254) (layer "B.Cu") (net 6))
+  (segment (start 167.64 75.184) (end 166.824 76) (width 0.4) (layer "B.Cu") (net 6))
   (segment (start 138 61.1) (end 138.7 60.4) (width 0.5) (layer "B.Cu") (net 6))
   (segment (start 138.7 60.4) (end 142.6 60.4) (width 0.5) (layer "B.Cu") (net 6))
-  (segment (start 179.832 80.772) (end 179.832 82.804) (width 0.254) (layer "B.Cu") (net 6))
+  (segment (start 179.832 80.772) (end 179.832 82.804) (width 0.4) (layer "B.Cu") (net 6))
   (segment (start 177.48 83.57) (end 177.48 88.3) (width 0.5) (layer "B.Cu") (net 6))
-  (segment (start 179.832 82.804) (end 179.086 83.55) (width 0.254) (layer "B.Cu") (net 6))
+  (segment (start 179.832 82.804) (end 179.086 83.55) (width 0.4) (layer "B.Cu") (net 6))
   (segment (start 134.3 65.45) (end 136.65 65.45) (width 0.4) (layer "B.Cu") (net 6))
   (segment (start 138 64.1) (end 138 61.1) (width 0.5) (layer "B.Cu") (net 6))
-  (segment (start 176.3 76) (end 175.484 75.184) (width 0.254) (layer "B.Cu") (net 6))
-  (segment (start 153.815 74.567) (end 153.815 70.8) (width 0.254) (layer "B.Cu") (net 6))
-  (segment (start 166.824 76) (end 155.248 76) (width 0.254) (layer "B.Cu") (net 6))
+  (segment (start 176.3 76) (end 175.484 75.184) (width 0.4) (layer "B.Cu") (net 6))
+  (segment (start 153.815 74.567) (end 153.815 70.8) (width 0.4) (layer "B.Cu") (net 6))
+  (segment (start 166.824 76) (end 155.248 76) (width 0.4) (layer "B.Cu") (net 6))
   (segment (start 177.55 83.6) (end 177.5 83.55) (width 0.254) (layer "B.Cu") (net 6))
   (segment (start 142.6 60.4) (end 142.9 60.7) (width 0.5) (layer "B.Cu") (net 6))
-  (segment (start 155.248 76) (end 153.815 74.567) (width 0.254) (layer "B.Cu") (net 6))
-  (segment (start 179.086 83.55) (end 177.5 83.55) (width 0.254) (layer "B.Cu") (net 6))
+  (segment (start 155.248 76) (end 153.815 74.567) (width 0.4) (layer "B.Cu") (net 6))
+  (segment (start 179.086 83.55) (end 177.5 83.55) (width 0.4) (layer "B.Cu") (net 6))
   (segment (start 136.65 65.45) (end 138 64.1) (width 0.5) (layer "B.Cu") (net 6))
   (segment (start 144.2 70.8) (end 153.815 70.8) (width 0.5) (layer "B.Cu") (net 6))
