File: PCB/PCB_VuilBak_Kicad/PCB_VuilBak.kicad_sch (KiCad schematic)
At the start: 15 parts

Commit message: verder gewerkt aan PCB
Parts:
- added R? (x2): 10k, symbol Device:R
- added R?: 499, symbol Device:R
- added S? (x2): DTE6, switch-misc_DTE6, symbol switch-misc:DTE6
Connections:
- net GND: now also S?.1 (S), S?.2 (S), S?.3 (P), S?.4 (P)
- net at U?.23 (GPIO0): now also R?.1, S?.3 (P), S?.4 (P)
- net RX: now reaches U?.40 (U0RXD)
- net at U?.41 (U0TXD): now also R?.1
- net at U?.9 (CHIP_PU): now also R?.1, S?.1 (S), S?.2 (S)
- net Voeding voor flash renamed voeding voor flash (ongv. 3.3 V)
- new net TX: R?.2
- new net reset input 3.3V: R?.2
- new net set input 3.3V: R?.2
Other:
- note added: "Analog power input circuit zie design guidlines"
- note added: "Best hoger dan 3V (eerder 3.3V)"
- note added: "pins 40/41 zijn voor uart"
- moved on the sheet: C?, L?, R?, U?

Commit message: pcb schema updated
Parts:
- removed C?: 1u, symbol Device:C
- added U?: level_shifter, symbol Onze_Bib:level_shifter
- added U?: TCA9548A_I2C_Multiplexer, symbol Onze_Bib:TCA9548A_I2C_Multiplexer
- added U? (x2): Step_down_buck, symbol Onze_Bib:Step_down_buck
Connections:
- net Analog power input (2.3-3.6V) is gone; now on net 3.3V: C?.1, C?.1, C?.1, C?.1, C?.1, C?.2, C?.2, L?.1, U?.1 (VDDA), U?.43 (VDDA), U?.46 (VDDA)
- net reset input 3.3V is gone; now on net 3.3V: R?.2
- net set input 3.3V is gone; now on net 3.3V: R?.2
- net GND: now also U?.2 (GND), U?.3 (IN+), U?.3 (IN+), U?.4 (GND), U?.6 (A0), U?.6 (OUT+), U?.6 (OUT+), U?.7 (A1), U?.8 (A2), U?.9 (GND)
- net SCL_ESP: now reaches U?.39 (GPIO22)
- net SCL_ESP: now also U?.11 (LV2)
- net SDA_ESP: now reaches U?.42 (GPIO21)
- net SDA_ESP: now also U?.12 (LV1)
- net 1.8~3.6V renamed 3.3V
- net 3.3V: now also U?.1 (Vin), U?.10 (LV), U?.2 (IN-)
- net voeding voor flash (ongv. 3.3 V): no longer names the net of U?.26 (VDD_SDIO)
- new net 12V_IN: U?.7 (OUT-), U?.7 (OUT-)
- new net 5V: U?.2 (IN-), U?.3 (HV)
- new net SC2: U?.14 (SC2)
- new net SC3: U?.16 (SC3)
- new net SC4: U?.18 (SC4)
- new net SC5: U?.20 (SC5)
- new net SC6: U?.22 (SC6)
- new net SC7: U?.24 (SC7)
- new net SCL_Mux: U?.2 (HV2), U?.4 (SCL)
- new net SD2: U?.13 (SD2)
- new net SD3: U?.15 (SD3)
- new net SD4: U?.17 (SD4)
- new net SD5: U?.19 (SD5)
- new net SD6: U?.21 (SD6)
- new net SD7: U?.23 (SD7)
- new net SDA_mux: U?.1 (HV1), U?.3 (SDA)
Other:
- note added: "1.8~3.6V"
- note added: "12V voedingsspanning"
- note added: "3.3V output"
- note added: "Analog power input (2.3-3.6V)"
- note added: "Deze pins naar output om esp te programmeren"
- note added: "MUX channel (1)"
- note added: "MUX channel (2)"
- note added: "MUX channel (3)"
- note added: "MUX channel (4)"
- note added: "MUX channel (5)"
- note added: "MUX channel (6)"
- note added: "Moet volgens de datasheet"
- note added: "UART pins"
- note added: "Vin (3.3V)"
- note added: "reset input 3.3V"
- note added: "set input 3.3V"
- note removed: "Analog power input circuit zie design guidlines"
- moved on the sheet: C?, L?, R?, S?, U?

Commit message: update pcb-schema
Parts:
- added J?: Conn_01x12_Female, symbol Connector:Conn_01x12_Female
- added J?: Conn_01x04_Male, symbol Connector:Conn_01x04_Male
- added J?: Conn_01x13_Male, symbol Connector:Conn_01x13_Male
Connections:
- net 12V_IN: now also J?.2 (Pin_2)
- net 3.3V: now also J?.1 (Pin_1)
- net 5V: now also J?.1 (Pin_1), J?.5 (Pin_5), J?.9 (Pin_9)
- net GND: now also J?.12 (Pin_12), J?.4 (Pin_4), J?.4 (Pin_4), J?.8 (Pin_8)
- net RX: now also J?.3 (Pin_3)
- net SC2: now also J?.2 (Pin_2)
- net SC3: now also J?.7 (Pin_7)
- net SC4: now also J?.11 (Pin_11)
- net SD2: now also J?.3 (Pin_3)
- net SD3: now also J?.6 (Pin_6)
- net SD4: now also J?.10 (Pin_10)
- net TX: now also J?.2 (Pin_2)
- net GPIO25: now reaches U?.14 (GPIO25)
- net GPIO25: now also J?.3 (Pin_3)
- net GPIO26: now reaches U?.15 (GPIO26)
- net GPIO26: now also J?.4 (Pin_4)
- net GPIO27: now reaches U?.16 (GPIO27)
- net GPIO27: now also J?.5 (Pin_5)
- net GPIO2: now reaches U?.22 (GPIO2)
- net GPIO2: now also J?.6 (Pin_6)
- net GPIO4: now reaches U?.24 (GPIO4)
- net GPIO4: now also J?.7 (Pin_7)
- net GPIO 16: now reaches U?.25 (GPIO16)
- net GPIO 16: now also J?.8 (Pin_8)
- net GPIO 17: now reaches U?.27 (GPIO17)
- net GPIO 17: now also J?.9 (Pin_9)
- net GPIO 5: now reaches U?.34 (GPIO5)
- net GPIO 5: now also J?.10 (Pin_10)
- net GPIO 18: now reaches U?.35 (GPIO18)
- net GPIO 18: now also J?.11 (Pin_11)
- net GPIO 23: now reaches U?.36 (GPIO23)
- net GPIO 23: now also J?.12 (Pin_12)
- net GPIO 19: now reaches U?.38 (GPIO19)
- net GPIO 19: now also J?.13 (Pin_13)
- net SCL_Mux renamed SCL_LCD
- net SDA_mux renamed SDA_LCD
Other:
- note added: "Dit moet vervangen worden door inhoud IC"
- note added: "ESP 32"
- note added: "LEVEL SHIFTER VOOR VERSTERKING SIGNALEN"
- note added: "MULTIPLEXER"
- note added: "POWER CIRCUIT"
- note added: "Pins voor I2C communicatie met LCD"
- note added: "voor gewichtsensoren"
- note removed: "3.3V output"
- moved on the sheet: C?, L?, R?, S?, U?

Commit message: update pcb
Parts:
- removed C? (x4): 0.1u, symbol Device:C
- removed C? (x2): 10u, symbol Device:C
- removed C? (x2): 3.3n, symbol Device:C
- removed C?: 100p, symbol Device:C
- removed C? (x2): 1u, symbol Device:C
- removed J?: Conn_01x12_Female, symbol Connector:Conn_01x12_Female
- removed J?: Conn_01x04_Male, symbol Connector:Conn_01x04_Male
- removed J?: Conn_01x13_Male, symbol Connector:Conn_01x13_Male
- removed L?: 2n, symbol Device:L
- removed R?: 20k, symbol Device:R
- removed R? (x2): 10k, symbol Device:R
- removed R?: 499, symbol Device:R
- removed S? (x2): DTE6, switch-misc_DTE6, symbol switch-misc:DTE6
- removed U?: level_shifter, symbol Onze_Bib:level_shifter
- removed U?: TCA9548A_I2C_Multiplexer, symbol Onze_Bib:TCA9548A_I2C_Multiplexer
- removed U?: ESP32, symbol Onze_Bib:ESP32
- removed U? (x2): Step_down_buck, symbol Onze_Bib:Step_down_buck
- added C1: 10u, Capacitor_SMD:C_0805_2012Metric, symbol Device:C
- added C2: 1u, Capacitor_SMD:C_0805_2012Metric, symbol Device:C
- added C3, C5: 10u, Capacitor_SMD:C_0805_2012Metric, symbol Device:C_Polarized
- added C4: 22u, Capacitor_SMD:C_0805_2012Metric, symbol Device:C
- added C6, C7: 0.1u, Capacitor_SMD:C_0805_2012Metric, symbol Device:C
- added Q1, Q2: 2N7002, Package_TO_SOT_SMD:SOT-23, symbol Transistor_FET:2N7002
- added R1, R11, R12, R13, R2, R3, R4, R5, R6, R7, R8: 10k, Capacitor_SMD:C_0805_2012Metric, symbol Device:R
- added S1, S2: DTE6, switch:SW_1571527-1, symbol switch-misc:DTE6
- added U1: micro_usb, micro_usb:GCT_USB3090-XX-X_REVE, symbol Onze_Bib:micro_usb
- added U2: AMS1117-3.3, Package_TO_SOT_SMD:SOT-223-3_TabPin2, symbol Regulator_Linear:AMS1117-3.3
- added U3: TCA9548A_I2C_Multiplexer, TCA:SOP65P640X120-24N, symbol Onze_Bib:TCA9548A_I2C_Multiplexer
- added U4: esp_wroom_32, Nieuwe map (2):MODULE_ESP32-WROOM-32, symbol Onze_Bib:esp_wroom_32
- added X1, X10, X2, X3, X4, X7, X8, X9: DG3XX-04-3.5, pins:PinHeader_1x04_P2.54mm_Vertical, symbol degson:DG3XX-04-3.5
- added X11, X12, X13: DG3XX-02-3.5, pins:PinHeader_1x02_P2.54mm_Vertical, symbol degson:DG3XX-02-3.5
- added X5: DG3XX-03-3.5, pins:PinHeader_1x03_P2.54mm_Vertical, symbol degson:DG3XX-03-3.5
- added X6: DG3XX-07-3.5, pins:PinHeader_1x07_P2.54mm_Vertical, symbol degson:DG3XX-07-3.5
Connections:
- net 3.3V: now also C1.2, C4.2, C5.1, C6.2, Q1.1 (G), Q2.1 (G), R1.2, R2.2, R3.1, R4.1, R7.2, R8.2, U2.2 (VO), U3.24 (VCC), U4.2 (3V3), X1.4 (KL), X11.1 (KL), X12.1 (KL), X13.1 (KL)
- net 5V: now also C3.1, R5.1, R6.1, U1.1 (VCC), U2.3 (VI), X10.1 (KL), X2.4 (KL), X3.4 (KL), X4.1 (KL), X5.1 (KL), X7.1 (KL), X8.1 (KL), X9.1 (KL)
- net GND: now also C1.1, C2.2, C3.2, C4.1, C5.2, C6.1, C7.1, R11.2, R12.2, R13.2, S1.3 (P), S1.4 (P), S2.1 (S), S2.2 (S), U1.5 (GND), U2.1 (GND), U3.1 (A0), U3.12 (GND), U3.2 (A1), U3.21 (A2), U4.1 (GND), U4.15 (GND), U4.38 (GND), U4.39_1 (GND), U4.39_10 (GND), U4.39_11 (GND), U4.39_12 (GND), U4.39_13 (GND), U4.39_14 (GND), U4.39_15 (GND), U4.39_16 (GND), U4.39_17 (GND), U4.39_18 (GND), U4.39_19 (GND), U4.39_2 (GND), U4.39_20 (GND), U4.39_21 (GND), U4.39_3 (GND), U4.39_4 (GND), U4.39_5 (GND), U4.39_6 (GND), U4.39_7 (GND), U4.39_8 (GND), U4.39_9 (GND), X1.1 (KL), X10.4 (KL), X2.1 (KL), X3.1 (KL), X4.4 (KL), X5.2 (KL), X7.4 (KL), X8.4 (KL), X9.4 (KL)
- net GPIO 16: now also U4.27 (IO16), X6.5 (KL)
- net GPIO 17: now also U4.28 (IO17), X6.4 (KL)
- net GPIO 18: now also U4.30 (IO18), X6.2 (KL)
- net GPIO 19: now also U4.31 (IO19), X6.1 (KL)
- net GPIO 23: now also U4.37 (IO23), X5.3 (KL)
- net GPIO 5: now also U4.29 (IO5), X6.3 (KL)
- net GPIO2: now also U4.24 (IO2), X6.7 (KL)
- net GPIO25: now also R11.1, U4.10 (IO25), X11.2 (KL)
- net GPIO26: now also U4.11 (IO26), X2.2 (KL)
- net GPIO27: now also U4.12 (IO27), X2.3 (KL)
- net GPIO4: now also U4.26 (IO4), X6.6 (KL)
- net RX: now also U4.34 (RXD0), X1.3 (KL)
- net SC5: now also U3.16 (SC5), X7.2 (KL)
- net SC6: now also U3.18 (SC6), X8.2 (KL)
- net SC7: now also U3.20 (SC7), X9.2 (KL)
- net SCL_ESP: now also Q1.2 (S), R3.2, U4.36 (IO22)
- net SD5: now also U3.15 (SD5), X7.3 (KL)
- net SD6: now also U3.17 (SD6), X8.3 (KL)
- net SD7: now also U3.19 (SD7), X9.3 (KL)
- net SDA_ESP: now also Q2.2 (S), R4.2, U4.33 (IO21)
- net TX: now also U4.35 (TXD0), X1.2 (KL)
- new net: R8.1, S2.3 (P), S2.4 (P), U4.25 (IO0)
- new net: C2.1, C7.2, R7.1, S1.1 (S), S1.2 (S), U4.3 (EN)
- new net GPIO12: U4.14 (IO12), X4.3 (KL)
- new net GPIO13: U4.16 (IO13), X3.3 (KL)
- new net GPIO14: U4.13 (IO14), X4.2 (KL)
- new net GPIO15: U4.23 (IO15), X3.2 (KL)
- new net GPIO32: R12.1, U4.8 (IO32), X12.2 (KL)
- new net GPIO33: R13.1, U4.9 (IO33), X13.2 (KL)
- new net SCL_Mux: Q1.3 (D), R1.1, R5.2, U3.22 (SCL), X10.3 (KL)
- new net SDA_mux: Q2.3 (D), R2.1, R6.2, U3.23 (SDA), X10.2 (KL)
Other:
- note added: "Buttons"
- note added: "I/O"
- note added: "RFID 1"
- note added: "RFID 2"
- note added: "RFID 3"
- note removed: "1.8~3.6V"
- note removed: "12V voedingsspanning"
- note removed: "Analog power input (2.3-3.6V)"
- note removed: "Best hoger dan 3V (eerder 3.3V)"
- note removed: "Deze pins naar output om esp te programmeren"
- note removed: "Dit moet vervangen worden door inhoud IC"
- note removed: "MUX channel (1)"
- note removed: "MUX channel (2)"
- note removed: "MUX channel (3)"
- note removed: "Moet volgens de datasheet"
- note removed: "Vin (3.3V)"
- note removed: "Voeding voor CPU"
- note removed: "Voeding voor RTC"
- note removed: "pins 40/41 zijn voor uart"
- note removed: "voor gewichtsensoren"

Commit message: Update pcb
Parts:
- S1, S2: value DTE6 -> (none); footprint switch:SW_1571527-1 -> (none)
Changed lines of the file:
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@@
       (effects (font (size 1.27 1.27)) hide)
     )
-    (pin "3")
+    (pin "1")
+    (pin "2")
+    (pin "3")
+    (pin "4")
   )
   (symbol (lib_id "Onze_Bib:esp_wroom_32") (at 242.57 60.96 0) (unit 1)
@@
       (effects (font (size 1.27 1.27)) hide)
     )
-    (pin "3")
+    (pin "1")
+    (pin "2")
+    (pin "3")
+    (pin "4")
   )
   (symbol (lib_id "switch-misc:DTE6") (at 182.88 72.39 270) (unit 1)
@@
       (effects (font (size 1.143 1.143)))
     )
-    (property "Value" "DTE6" (id 1) (at 182.88 63.5 90)
+    (property "Value" "" (id 1) (at 182.88 63.5 90)
       (effects (font (size 1.143 1.143)))
     )
-    (property "Footprint" "switch:SW_1571527-1" (id 2) (at 186.69 73.152 0)
+    (property "Footprint" "" (id 2) (at 186.69 73.152 0)
       (effects (font (size 0.508 0.508)) hide)
     )
@@
       (effects (font (size 1.27 1.27)) hide)
     )
-    (pin "2")
+    (pin "1")
+    (pin "2")
+    (pin "3")
+    (pin "4")
   )
   (symbol (lib_id "power:GND") (at 269.24 41.91 180) (unit 1)
@@
       (effects (font (size 1.27 1.27)) hide)
     )
+    (pin "1")
     (pin "2")
   )
@@
       (effects (font (size 1.27 1.27)) hide)
     )
-    (pin "3")
+    (pin "1")
+    (pin "2")
+    (pin "3")
+    (pin "4")
   )
   (symbol (lib_id "degson:DG3XX-02-3.5") (at 337.82 190.5 0) (unit 1)
@@
     )
     (pin "1")
+    (pin "2")
   )
   (symbol (lib_id "power:GND") (at 281.94 41.91 180) (unit 1)
@@
       (effects (font (size 1.27 1.27)) hide)
     )
+    (pin "1")
+    (pin "2")
+    (pin "3")
     (pin "4")
   )
@@
       (effects (font (size 1.27 1.27)) hide)
     )
-    (pin "3")
+    (pin "1")
+    (pin "2")
+    (pin "3")
+    (pin "4")
   )
   (symbol (lib_id "Device:R") (at 50.8 59.69 0) (unit 1)
@@
     )
     (pin "1")
+    (pin "2")
+    (pin "3")
+    (pin "4")
+    (pin "5")
+    (pin "6")
+    (pin "7")
   )
   (symbol (lib_id "degson:DG3XX-04-3.5") (at 187.96 205.74 0) (unit 2)
@@
       (effects (font (size 1.27 1.27)) hide)
     )
-    (pin "2")
+    (pin "1")
+    (pin "2")
+    (pin "3")
+    (pin "4")
   )
   (symbol (lib_id "degson:DG3XX-04-3.5") (at 259.08 228.6 0) (unit 4)
@@
       (effects (font (size 1.27 1.27)) hide)
     )
+    (pin "1")
+    (pin "2")
+    (pin "3")
     (pin "4")
   )
@@
     )
     (pin "1")
+    (pin "2")
   )
   (symbol (lib_id "power:GND") (at 110.49 140.97 0) (unit 1)
@@
       (effects (font (size 1.27 1.27)) hide)
     )
+    (pin "1")
+    (pin "2")
+    (pin "3")
+    (pin "4")
+    (pin "5")
+    (pin "6")
     (pin "7")
   )
@@
       (effects (font (size 1.27 1.27)) hide)
     )
+    (pin "1")
+    (pin "2")
     (pin "3")
   )
@@
       (effects (font (size 1.27 1.27)) hide)
     )
+    (pin "1")
     (pin "2")
   )
@@
       (effects (font (size 1.27 1.27)) hide)
     )
-    (pin "4")
+    (pin "1")
+    (pin "2")
+    (pin "3")
+    (pin "4")
+    (pin "5")
+    (pin "6")
+    (pin "7")
   )
   (symbol (lib_id "degson:DG3XX-04-3.5") (at 259.08 248.92 0) (unit 4)
@@
       (effects (font (size 1.27 1.27)) hide)
     )
+    (pin "1")
+    (pin "2")
+    (pin "3")
     (pin "4")
   )
@@
     )
     (pin "1")
+    (pin "2")
+    (pin "3")
+    (pin "4")
   )
   (symbol (lib_id "Device:R") (at 46.99 111.76 0) (unit 1)
@@
       (effects (font (size 1.27 1.27)) hide)
     )
+    (pin "1")
+    (pin "2")
+    (pin "3")
+    (pin "4")
+    (pin "5")
     (pin "6")
+    (pin "7")
   )
   (symbol (lib_id "degson:DG3XX-04-3.5") (at 187.96 203.2 0) (unit 1)
@@
     )
     (pin "1")
+    (pin "2")
+    (pin "3")
+    (pin "4")
   )
   (symbol (lib_id "degson:DG3XX-04-3.5") (at 259.08 256.54 0) (unit 3)
@@
       (effects (font (size 1.27 1.27)) hide)
     )
-    (pin "3")
+    (pin "1")
+    (pin "2")
+    (pin "3")
+    (pin "4")
   )
   (symbol (lib_id "degson:DG3XX-04-3.5") (at 187.96 200.66 0) (unit 4)
@@
       (effects (font (size 1.27 1.27)) hide)
     )
+    (pin "1")
+    (pin "2")
+    (pin "3")
     (pin "4")
   )
@@
       (effects (font (size 1.27 1.27)) hide)
     )
+    (pin "1")
+    (pin "2")
+    (pin "3")
     (pin "4")
   )
@@
       (effects (font (size 1.27 1.27)) hide)
     )
-    (pin "2")
+    (pin "1")
+    (pin "2")
+    (pin "3")
+    (pin "4")
+    (pin "5")
+    (pin "6")
+    (pin "7")
   )
   (symbol (lib_id "Onze_Bib:micro_usb") (at 49.53 168.91 0) (unit 1)
@@
     )
     (pin "1")
+    (pin "2")
+    (pin "3")
+    (pin "4")
   )
   (symbol (lib_id "degson:DG3XX-03-3.5") (at 255.27 209.55 0) (unit 2)
@@
       (effects (font (size 1.27 1.27)) hide)
     )
-    (pin "2")
+    (pin "1")
+    (pin "2")
+    (pin "3")
   )
   (symbol (lib_id "degson:DG3XX-04-3.5") (at 259.08 241.3 0) (unit 1)
@@
     )
     (pin "1")
+    (pin "2")
+    (pin "3")
+    (pin "4")
   )
   (symbol (lib_id "degson:DG3XX-04-3.5") (at 259.08 233.68 0) (unit 2)
@@
       (effects (font (size 1.27 1.27)) hide)
     )
-    (pin "2")
+    (pin "1")
+    (pin "2")
+    (pin "3")
+    (pin "4")
   )
   (symbol (lib_id "power:GND") (at 261.62 130.81 0) (unit 1)
@@
       (effects (font (size 1.27 1.27)) hide)
     )
-    (pin "3")
+    (pin "1")
+    (pin "2")
+    (pin "3")
+    (pin "4")
+    (pin "5")
+    (pin "6")
+    (pin "7")
   )
   (symbol (lib_id "Device:R") (at 339.09 213.36 0) (mirror y) (unit 1)
@@
       (effects (font (size 1.27 1.27)) hide)
     )
-    (pin "3")
+    (pin "1")
+    (pin "2")
+    (pin "3")
+    (pin "4")
   )
   (symbol (lib_id "power:GND") (at 172.72 203.2 270) (unit 1)
@@
       (effects (font (size 1.27 1.27)) hide)
     )
-    (pin "2")
+    (pin "1")
+    (pin "2")
+    (pin "3")
+    (pin "4")
   )
   (symbol (lib_id "Regulator_Linear:AMS1117-3.3") (at 78.74 199.39 0) (unit 1)
@@
     )
     (pin "1")
+    (pin "2")
+    (pin "3")
+    (pin "4")
   )
   (symbol (lib_id "Device:C") (at 204.47 76.2 0) (unit 1)
@@
     )
     (pin "1")
+    (pin "2")
+    (pin "3")
+    (pin "4")
   )
   (symbol (lib_id "degson:DG3XX-03-3.5") (at 255.27 207.01 0) (unit 1)
@@
     )
     (pin "1")
+    (pin "2")
+    (pin "3")
   )
   (symbol (lib_id "degson:DG3XX-04-3.5") (at 259.08 223.52 0) (unit 2)
@@
       (effects (font (size 1.27 1.27)) hide)
     )
-    (pin "2")
+    (pin "1")
+    (pin "2")
+    (pin "3")
+    (pin "4")
   )
   (symbol (lib_id "power:GND") (at 173.99 72.39 270) (unit 1)
@@
       (effects (font (size 1.27 1.27)) hide)
     )
+    (pin "1")
+    (pin "2")
+    (pin "3")
     (pin "4")
   )
@@
       (effects (font (size 1.27 1.27)) hide)
     )
-    (pin "3")
+    (pin "1")
+    (pin "2")
+    (pin "3")
+    (pin "4")
   )
   (symbol (lib_id "degson:DG3XX-04-3.5") (at 259.08 220.98 0) (unit 1)
@@
     )
     (pin "1")
+    (pin "2")
+    (pin "3")
+    (pin "4")
   )
   (symbol (lib_id "degson:DG3XX-04-3.5") (at 259.08 243.84 0) (unit 2)
@@
       (effects (font (size 1.27 1.27)) hide)
     )
-    (pin "2")
+    (pin "1")
+    (pin "2")
+    (pin "3")
+    (pin "4")
   )
   (symbol (lib_id "power:GND") (at 63.5 207.01 0) (unit 1)
@@
       (effects (font (size 1.27 1.27)) hide)
     )
-    (pin "2")
+    (pin "1")
+    (pin "2")
+    (pin "3")
+    (pin "4")
   )
   (symbol (lib_id "degson:DG3XX-04-3.5") (at 259.08 238.76 0) (unit 4)
@@
       (effects (font (size 1.27 1.27)) hide)
     )
+    (pin "1")
+    (pin "2")
+    (pin "3")
     (pin "4")
   )
@@
       (effects (font (size 1.27 1.27)) hide)
     )
+    (pin "1")
+    (pin "2")
+    (pin "3")
     (pin "4")
   )
@@
     )
     (pin "1")
+    (pin "2")
   )
   (symbol (lib_id "power:GND") (at 245.11 228.6 270) (unit 1)
@@
       (effects (font (size 1.143 1.143)))
     )
-    (property "Value" "DTE6" (id 1) (at 293.37 63.5 90)
+    (property "Value" "" (id 1) (at 293.37 63.5 90)
       (effects (font (size 1.143 1.143)))
     )
-    (property "Footprint" "switch:SW_1571527-1" (id 2) (at 297.18 73.152 0)
+    (property "Footprint" "" (id 2) (at 297.18 73.152 0)
       (effects (font (size 0.508 0.508)) hide)
     )
@@
       (effects (font (size 1.27 1.27)) hide)
     )
+    (pin "1")
     (pin "2")
   )
@@
       (effects (font (size 1.27 1.27)) hide)
     )
-    (pin "3")
+    (pin "1")
+    (pin "2")
+    (pin "3")
+    (pin "4")
   )
   (symbol (lib_id "power:GND") (at 48.26 91.44 180) (unit 1)
@@
       (effects (font (size 1.27 1.27)) hide)
     )
-    (pin "2")
+    (pin "1")
+    (pin "2")
+    (pin "3")
+    (pin "4")
   )
   (symbol (lib_id "degson:DG3XX-07-3.5") (at 256.54 195.58 0) (unit 5)
@@
       (effects (font (size 1.27 1.27)) hide)
     )
+    (pin "1")
+    (pin "2")
+    (pin "3")
+    (pin "4")
     (pin "5")
+    (pin "6")
+    (pin "7")
   )
   (symbol (lib_id "degson:DG3XX-04-3.5") (at 187.96 193.04 0) (unit 1)
@@
     )
     (pin "1")
+    (pin "2")
+    (pin "3")
+    (pin "4")
   )
   (sheet_instances
@@
     )
     (path "/10375731-a3f1-470b-9c22-dc9e8252c951"
-      (reference "S1") (unit 1) (value "DTE6") (footprint "switch:SW_1571527-1")
+      (reference "S1") (unit 1) (value "DTE6") (footprint "1-1825910-4:TE_1-1825910-4")
     )
     (path "/e5027579-37e1-48bd-97c5-4fef51856c45"
-      (reference "S2") (unit 1) (value "DTE6") (footprint "switch:SW_1571527-1")
+      (reference "S2") (unit 1) (value "DTE6") (footprint "1-1825910-4:TE_1-1825910-4")
     )
     (path "/7c0f2ca1-78c8-4baf-b3d3-3419aa300dae"

Commit message: update pcb
Parts:
- removed Q1, Q2: 2N7002, Package_TO_SOT_SMD:SOT-23, symbol Transistor_FET:2N7002
- removed U1: micro_usb, micro_usb:GCT_USB3090-XX-X_REVE, symbol Onze_Bib:micro_usb
- removed X7, X8, X9: DG3XX-04-3.5, pins:PinHeader_1x04_P2.54mm_Vertical, symbol degson:DG3XX-04-3.5
- added C8: 10u, Capacitor_SMD:C_0805_2012Metric, symbol Device:C
- added Q1, Q2: BSS138, Package_TO_SOT_SMD:SOT-23, symbol Transistor_FET:BSS138
- added R9: 10k, Capacitor_SMD:C_0805_2012Metric, symbol Device:R
- added U1: micro, micro_usb_2:MOLEX_105017-1001, symbol Onze_Bib:micro
- added X7, X8, X9: DG3XX-05-3.5, pins:PinHeader_1x05_P2.54mm_Vertical, symbol degson:DG3XX-05-3.5
- S1, S2: value (none) -> DTE6; footprint (none) -> knop:TE_1-1825910-4
Connections:
- net 3.3V: now also X2.4 (KL), X3.4 (KL), X4.1 (KL), C8.2, Q1.1 (G), Q2.1 (G); no longer C1.2, R1.2, R2.2, U3.24 (VCC)
- net 5V: now also C1.2, R1.2, R2.2, U3.24 (VCC), R9.1, U1.1, X7.1 (KL), X8.1 (KL), X9.1 (KL); no longer X2.4 (KL), X3.4 (KL), X4.1 (KL)
- net GND: now also C8.1, U1.5, U1.S1 (SHIELD), U1.S2 (SHIELD), U1.S3 (SHIELD), U1.S4 (SHIELD), U1.S5 (SHIELD), U1.S6 (SHIELD), X7.5 (KL), X8.5 (KL), X9.5 (KL)
- net GPIO 16: now also X7.4 (KL)
- net GPIO2: now also X9.4 (KL)
- net GPIO4: now also X8.4 (KL)
- net SC5: now also X7.2 (KL)
- net SC6: now also X8.2 (KL)
- net SC7: now also X9.2 (KL)
- net SCL_ESP: now also Q1.2 (S)
- net SCL_Mux: now also Q1.3 (D)
- net SD5: now also X7.3 (KL)
- net SD6: now also X8.3 (KL)
- net SD7: now also X9.3 (KL)
- net SDA_ESP: now also Q2.2 (S)
- net SDA_mux: now also Q2.3 (D)
- net at U3.3 (~{RESET}): now also R9.2
Other:
- note added: "Boot input 3.3V"
- note added: "Enable input 3.3V"
- note added: "Gewichtsensor (1)"
- note added: "Gewichtsensor (2)"
- note added: "Gewichtsensor (3)"
- note added: "luidspreker"
- note added: "reset active high"
- note removed: "reset input 3.3V"
- note removed: "set input 3.3V"
- moved on the sheet: C4, C6

Commit message: update schema
update schema voor documentatie
Other:
- note added: "ESP32-WROOM-32E"
- note removed: "ESP 32"
Changed lines of the file:
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@@
     (effects (font (size 1.27 1.27)) (justify left bottom))
   )
-  (text "ESP 32" (at 140.97 33.02 0)
+  (text "ESP32-WROOM-32E" (at 168.91 45.72 0)
     (effects (font (size 1.9 1.9) (thickness 0.4) bold italic) (justify left bottom))
   )
